Commit message: Minor changes.

File: tbotsim/script_build config/urdf/tetherbot.urdf (robot description, URDF)
Before this commit: robot tetherbot0, 120 links, 119 joints
Links:
- added link rectanglewrenchset0
- added link tetherforceset0
Joints:
- added joint map_to_tetherforceset0: type fixed, parent map, child tetherforceset0, origin xyz=0.0 0.0 0.0 rpy=0.0 -0.0 0.0
- added joint platform0_to_rectanglewrenchset0: type fixed, parent platform0, child rectanglewrenchset0, origin xyz=0.0 0.0 0.0 rpy=0.0 -0.0 0.0
